File: SimpleFC/IMU.sch (KiCad schematic (older format))
At the start: 26 parts, among them J8 UFL, U12 NEO-M8, U2 MAG3110, U3 ICM-20689, U4 MS5611

Commit message: Refactor SimpleFC schematics with latest KiCAD libraries.
Parts:
- removed U12: NEO-M8, LCC:UBX-LCC24, symbol ublox:NEO-M8
- added U12: NEO-M8N, LCC:UBX-LCC24, symbol RF_GPS:NEO-M8N
Connections:
- wire segments 130 -> 128
- no-connect marks 9 -> 10
Other:
- moved on the sheet: BT1, C42, D12, D13, J8, L3, R28, R29
