File: SimpleFC/Power.sch (KiCad schematic (older format))
At the start: 33 parts, among them J1 M02, Q1 AO3407A, U13 TPS79333, U5 MP2403, U6 SPX3819

Commit message: Refactor SimpleFC schematics with latest KiCAD libraries.
Parts:
- removed U13: TPS79333, STD_SMD:SOT-23-5, symbol LDO:TPS793xx
- removed U6: SPX3819, STD_SMD:SOT-23-5, symbol LDO:SPX3819
- added D4: 1A, STD_SMD:D_SOD-123, symbol Device:D_Schottky
- added U13: TPS79333-EP, Package_TO_SOT_SMD:SOT-23-5, symbol Regulator_Linear:TPS79333-EP
- added U6: SPX3819M5-L-3-3, Package_TO_SOT_SMD:SOT-23-5, symbol Regulator_Linear:SPX3819M5-L-3-3
- D15: renamed from D4; value 1A -> 3A; footprint STD_SMD:D_SOD-123 -> STD_SMD:D_SMA_Standard
Connections:
- net labels added: PRE5V
- wire segments 140 -> 142
Other:
- moved on the sheet: C30, C32, C43, C44, C45, D15
