File: SimpleFC/STM32F4.sch (KiCad schematic (older format))
At the start: 17 parts, among them U1 STM32F405RGTx, X1 25Mhz

Commit message: Refactor SimpleFC schematics with latest KiCAD libraries.
Parts:
- removed U1: STM32F405RGTx, Package_QFP:LQFP-64_10x10mm_P0.5mm, symbol SimpleFC-cache:STM32F405RGTx-MCU_ST_STM32
- added U1: STM32F405RGTx, Package_QFP:LQFP-64_10x10mm_P0.5mm, symbol MCU_ST_STM32F4:STM32F405RGTx
Connections:
- wire segments 121 -> 122
Other:
- moved on the sheet: C1, C2, C3, R1, R2, X1
