File: SimpleFC/Transceivers.sch (KiCad schematic (older format))
At the start: 15 parts, among them U10 74LVC1G86, U11 TJA1050, U8 74LVC1G86, U9 SN74LVC245APW

Commit message: Refactor SimpleFC schematics with latest KiCAD libraries.
Parts:
- removed U11: TJA1050, STD_SMD:SOIC-8_3.9x4.9mm_Pitch1.27mm, symbol bus-transceiver:TJA1050
- removed U9: SN74LVC245APW, Package_SSOP:TSSOP-20_4.4x6.5mm_P0.65mm, symbol LogicLevel:SN74LVC245APW
- added U11: TJA1050, Package_SO:SOIC-8_3.9x4.9mm_P1.27mm, symbol Interface_CAN_LIN:TJA1051T
- added U9: SN74LVC245APW, Package_SO:TSSOP-20_4.4x6.5mm_P0.65mm, symbol 74xx:74LS245
- U10, U8: symbol SimpleFC-cache:74LVC1G86-Logic_74xgxx -> SimpleFC-rescue:74LVC1G86-Logic_74xgxx-SimpleFC-cache
Connections:
- wire segments 94 -> 93
- no-connect marks 2 -> 1
Other:
- moved on the sheet: C39, R19
